Commit message: update sensor_kit

File: citac_sensor_kit_description/urdf/sensor_kit.xacro (robot description, xacro)
@@ -4,8 +4,10 @@
     <xacro:include filename="$(find velodyne_description)/urdf/VLP-16.urdf.xacro"/>
     <xacro:include filename="$(find vls_description)/urdf/VLS-128.urdf.xacro"/>
+    <xacro:include filename="$(find ouster_description)/urdf/OS1-64.urdf.xacro"/>
     <xacro:include filename="$(find camera_description)/urdf/monocular_camera.xacro"/>
     <xacro:include filename="$(find imu_description)/urdf/imu.xacro"/>
     <xacro:arg name="gpu" default="false"/>
-    <xacro:arg name="config_dir" default="$(find sample_sensor_kit_description)/config"/>
+    <!-- <xacro:arg name="config_dir" default="$(find sample_sensor_kit_description)/config"/> -->
+    <xacro:arg name="config_dir" default="$(find citac_sensor_kit_description)/config"/>
     <xacro:property name="sensor_kit_base_link" default="sensor_kit_base_link"/>
     <joint name="${sensor_kit_base_link}_joint" type="fixed">
@@ -20,5 +22,15 @@
     <xacro:property name="calibration" value="${xacro.load_yaml('$(arg config_dir)/sensor_kit_calibration.yaml')}"/>
     <!-- lidar -->
-    <xacro:VLS-128 parent="sensor_kit_base_link" name="velodyne_top" topic="/points_raw" hz="10" samples="220" gpu="$(arg gpu)">
+    <xacro:OS1-64 parent="sensor_kit_base_link" name="os_sensor" topic="/points" hz="10" samples="220" gpu="$(arg gpu)">
+      <origin
+        xyz="${calibration['sensor_kit_base_link']['os_sensor_base_link']['x']}
+             ${calibration['sensor_kit_base_link']['os_sensor_base_link']['y']}
+             ${calibration['sensor_kit_base_link']['os_sensor_base_link']['z']}"
+        rpy="${calibration['sensor_kit_base_link']['os_sensor_base_link']['roll']}
+             ${calibration['sensor_kit_base_link']['os_sensor_base_link']['pitch']}
+             ${calibration['sensor_kit_base_link']['os_sensor_base_link']['yaw']}"
+      />
+    </xacro:OS1-64>
+    <!-- <xacro:VLS-128 parent="sensor_kit_base_link" name="velodyne_top" topic="/points_raw" hz="10" samples="220" gpu="$(arg gpu)">
       <origin
         xyz="${calibration['sensor_kit_base_link']['velodyne_top_base_link']['x']}
@@ -29,5 +41,5 @@
              ${calibration['sensor_kit_base_link']['velodyne_top_base_link']['yaw']}"
       />
-    </xacro:VLS-128>
+    </xacro:VLS-128> -->
     <!-- camera -->
     <!-- <xacro:monocular_camera_macro
